Commit message: crown added (fet per tots)

File: src/my_robot_description/urdf/rubot/new_rubot_mecanum.urdf (robot description, URDF)
Before this commit: robot rubot, 9 links, 8 joints
Links:
- link part: geometry collision box size=0.05 0.05 0.025; visual mesh filename=file://$(find my_robot_description)/meshes/rubot/crown.STL scale=0.0004 0.0004 0.0004
